Commit message: feat: add gray and black materials for enhanced visual representation in URDF

File: hexapod_description/urdf/raspclaws_hexapod.urdf.xacro (robot description, xacro)
@@ -9,4 +9,10 @@
                         └── camera_link
   -->
+    <material name="gray">
+        <color rgba="0.5 0.5 0.5 1.0"/>
+    </material>
+        <material name="black">
+        <color rgba="0.0 0.0 0.0 1.0"/>
+    </material>
   <!-- ===================== -->
   <!-- Parameter (ANPASSEN!) -->
